File: proto_fpd_link/ice40.sch (KiCad schematic (older format))
At the start: 50 parts, among them J1 Conn_01x12, J101 Conn_02x05_Odd_Even, J102 Conn_01x18, J2 Conn_01x05, J3 Conn_01x19, J4 Conn_01x05, J5 Conn_01x01, J6 Conn_01x40_MountingPin, J7 Conn_01x01, U101 TLV71333PDBV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

Commit message: initial commit of ice40 programmer board
Parts:
- removed C101, C102, C105: 100n, Capacitor_SMD:C_0603_1608Metric, symbol ice40-rescue:C_Small-Device
- removed D101: BAT54C, Package_TO_SOT_SMD:SOT-23, symbol ice40-rescue:BAT54C-Diode
- removed J1: Conn_01x12, Connector_PinHeader_2.54mm:PinHeader_1x12_P2.54mm_Vertical, symbol Connector_Generic:Conn_01x12
- removed J102: Conn_01x18, Connector_PinHeader_2.54mm:PinHeader_1x18_P2.54mm_Vertical, symbol ice40-rescue:Conn_01x18-Connector_Generic
- removed J2, J4: Conn_01x05, Connector_PinHeader_2.54mm:PinHeader_1x05_P2.54mm_Vertical, symbol Connector_Generic:Conn_01x05
- removed J3: Conn_01x19, Connector_PinHeader_2.54mm:PinHeader_1x19_P2.54mm_Vertical, symbol Connector_Generic:Conn_01x19
- removed J5, J7: Conn_01x01, Connector_PinHeader_2.54mm:PinHeader_1x01_P2.54mm_Vertical, symbol Connector_Generic:Conn_01x01
- removed R104: NM, Resistor_SMD:R_0603_1608Metric, symbol ice40-rescue:R_Small-Device
- removed R111, R113, R2: 100R 1%, Resistor_SMD:R_0402_1005Metric, symbol ice40-rescue:R_Small-Device
- removed U101: TLV71333PDBV, Package_TO_SOT_SMD:SOT-23-5, symbol ice40-rescue:TLV71333PDBV-Regulator_Linear
- gave numbers to parts that had none: 1
Connections:
- net labels added: CLK_EDID, DATA_EDID, LED_EN, LED_PWM, LED_VCCS, RxCLK+, RxCLK-, Rxin0+, Rxin0-, Rxin1+, Rxin1-, Rxin2+, Rxin2-, VCCS, VEDID
- net labels removed: +5V, 1+, 1-, 12+, 12-, 2+, 2-, 4+, 4-, 6+, 6-, 7+, 7-, 9+, 9-
- wire segments 305 -> 256
- no-connect marks 3 -> 15
Other:
- note added: "12V (5-21V)"
- note added: "3V3"
- note added: "LED_GND"
- note added: "NOTE: Pin numbering swapped compared to display datasheet"
- note removed: "Bank 3 power supply\nShort Rxx for 3.3V operation"
- moved on the sheet: C103, C109, C112, C113, C114, C115, C116, J101, J6, R103, R105, R106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
